File: pcb_design/foc_controller/foc_controller.kicad_sch (KiCad schematic)
At the start: 18 parts, among them U4 AMS1117-3.3

Commit message: test pcb updated
Parts:
- removed TP1: TestPoint, TestPoint:TestPoint_Keystone_5010-5014_Multipurpose, symbol Connector:TestPoint
- added D?: LED_Small, symbol Device:LED_Small
- added J?: Conn_01x06_Socket, symbol Connector:Conn_01x06_Socket
- added JP?: V_batt, symbol Jumper:SolderJumper_2_Open
- added JP?: 3.3v, symbol Jumper:SolderJumper_2_Open
- added R?: 1k, symbol Device:R_Small
Connections:
- net +3.3V: now also D?.2 (A), JP?.1 (A)
- net +3V3: no longer U?.7 (VIN_AVDD)
- net GND: now also R?.1
- net +5V renamed +BATT
- net +BATT: now also JP?.1 (A)
- new net: JP?.2 (B), JP?.2 (B), U?.7 (VIN_AVDD)
- new net: D?.1 (K), R?.2
